File: Hardware/Design/small_led_driver.kicad_pcb (KiCad board)
At the start: 4 copper layers, 43.2 x 45.7 mm, 72 parts, among them J1 Conn_01x04_Male, J10 Conn_01x01_Male, J11 Conn_01x01_Male, J12 Conn_01x01_Male, J13 Conn_01x04_Male, J14 Conn_01x02_Male, J15 Conn_01x04_Male, J16 Conn_01x02_Male, J17 Conn_01x01_Male, J18 Conn_01x08_Male, J19 Conn_01x01_Male, J2 Conn_01x04_Male, J20 Conn_01x01_Male, J21 Conn_01x01_Male, J22 Conn_01x01_Male, J23 Conn_01x01_Male, J3 Conn_01x04_Male, J4 Conn_01x04_Male, J5 Conn_01x01_Male, J6 Conn_01x01_Male, J7 Conn_01x01_Male, J8 Conn_01x01_Male, J9 Conn_01x01_Male, Q1 BSS138, Q2 BSS138, SW1 SW_DIP_x01, U1 TXS0108EPW, U2 STM32L431RCTx, U3 LP5907MFX-3.3, Y1 ECS-480-8-36-RWN-TR, Y2 ECS-.327-9-1210-TR

Commit message: reorganize stm32 code 001
Routing:
- added copper zone on In1.Cu, net +3V3
- added copper zone on In1.Cu, net +5V
- added copper zone on In2.Cu, net GND1
- removed copper zone on PWR.Cu, net +3V3
- removed copper zone on PWR.Cu, net +5V
- removed copper zone on GND.Cu, net GND1
Other:
- net class Default removed
