File: Hardware/Design/opto_isolator.kicad_pcb (KiCad board)
At the start: 4 copper layers, 63.5 x 63.5 mm, 32 parts, among them J1 Conn_01x01_Male, J2 Conn_01x05_Male, J3 Conn_01x01_Male, U1 receiver_433MHz, U2 receiver_433MHz, U3 receiver_433MHz, U4 receiver_433MHz, U5 PS2501-4

Commit message: update based on testing of new level shifter
Routing:
- added copper zone on In2.Cu, net GND
- added copper zone on In1.Cu, net VCC
- removed copper zone on GND, net GND
- removed copper zone on PWR, net VCC
Other:
- net class Default removed
